File: soldering_station.kicad_sch (KiCad schematic)
At the start: 17 parts, among them J1 Barrel_Jack_Switch, J2 Conn_01x05, J6 USB, SW1 Rotary_Encoder_Switch_with_Mo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, U1 2.4inch_ST7789V_LCD

Commit message: Ready for review
Parts:
- removed R54: 3k3, Resistor_SMD:R_0402_1005Metric, symbol Device:R
- removed U1: 2.4inch_ST7789V_LCD, liebler_OPTO:2,4zoll lcd tft touch, symbol liebler_OPTO:2.4inch_ST7789V_LCD
- added BZ1: Buzzer, liebler_MECH:XDCR_CMT-7525-80-SMT-TR_handsolder, symbol liebler_MECH:Buzzer
- added C1: u1/35V, Capacitor_SMD:C_0805_2012Metric, symbol Device:C
- added C10, C11, C15, C21, C22, C23, C24, C25, C26, C27, C28, C29, C7, C8: u1, Capacitor_SMD:C_0201_0603Metric, symbol Device:C
- added C12, C9: 10u, Capacitor_SMD:C_0603_1608Metric, symbol Device:C
- added C13: 2n2, Capacitor_SMD:C_0201_0603Metric, symbol Device:C
- added C14, C17: 1u, Resistor_SMD:R_0402_1005Metric, symbol Device:C
- added C16: 22u, Capacitor_SMD:C_0603_1608Metric, symbol Device:C
- added C18: 10u/35V, Capacitor_SMD:C_0603_1608Metric, symbol Device:C
- added C19: 1u, Capacitor_SMD:C_0201_0603Metric, symbol Device:C
- added C2: 10u/35V, Capacitor_SMD:C_1206_3216Metric, symbol Device:C
- added C20: 22n, Capacitor_SMD:C_0201_0603Metric, symbol Device:C
- added C3: u1/16V, Capacitor_SMD:C_0201_0603Metric, symbol Device:C
- added C30, C31, C32: 10n, Capacitor_SMD:C_0201_0603Metric, symbol Device:C
- added C4: 56p, Capacitor_SMD:C_0201_0603Metric, symbol Device:C
- added C5, C6: 22u, Resistor_SMD:R_0805_2012Metric_Pad1.20x1.40mm_HandSolder, symbol Device:C
- added D10: ~, liebler_SEMICONDUCTORS:D_SOD-123_handsolder, symbol Device:D_Schottky
- added D11: 18V, liebler_SEMICONDUCTORS:D_SOD-123_handsolder, symbol Device:D_Zener
- added D12: LED, LED_SMD:LED_0805_2012Metric_Pad1.15x1.40mm_HandSolder, symbol Device:LED
- added D13, D9: D_Schottky, Diode_SMD:D_SMA, symbol Device:D_Schottky
- added H1, H2: MountingHole, MountingHole:MountingHole_3.2mm_M3, symbol Mechanical:MountingHole
- added J3: USB, liebler_CONN:GT-USB-7051A, symbol Connector:USB_C_Receptacle_USB2.0
- added J32: PROG, Connector_PinHeader_1.27mm:PinHeader_2x03_P1.27mm_Vertical_SMD, symbol Connector_Generic:Conn_02x03_Odd_Even
- added J5: EXT, Connector_PinHeader_2.54mm:PinHeader_1x05_P2.54mm_Vertical, symbol Connector_Generic:Conn_01x05
- added JP1: 20V, Jumper:SolderJumper-2_P1.3mm_Open_RoundedPad1.0x1.5mm, symbol Jumper:Jumper_2_Open
- added L1: 10uH, Inductor_SMD:L_Abracon_ASPI-0630LR, symbol Device:L
- added Q1: BC847, Package_TO_SOT_SMD:SOT-23, symbol Transistor_BJT:BC847
- added Q2: Q_PMOS_GDS, Package_DFN_QFN:PQFN-8-EP_6x5mm_P1.27mm_Generic, symbol Transistor_FET:Q_PMOS_GDS
- added Q3: MMBT2222A, Package_TO_SOT_SMD:SOT-23, symbol Transistor_BJT:MMBT2222A
- added Q4: BC847, Package_TO_SOT_SMD:SOT-23_Handsoldering, symbol Transistor_BJT:BC847
- added R1, R17, R21, R22, R23, R27, R47, R7: 10k, Resistor_SMD:R_0201_0603Metric, symbol Device:R
- added R10, R3, R6: 1k, Resistor_SMD:R_0201_0603Metric, symbol Device:R
- added R11: 4k7, Resistor_SMD:R_0805_2012Metric_Pad1.20x1.40mm_HandSolder, symbol Device:R
- added R12, R13, R18, R19, R20, R24, R28, R29, R4, R9: 3k3, Resistor_SMD:R_0201_0603Metric, symbol Device:R
- added R2: M1, Resistor_SMD:R_0201_0603Metric, symbol Device:R
- added R25: 5k1, Resistor_SMD:R_0201_0603Metric, symbol Device:R
- added R26, R30: 22R, Resistor_SMD:R_0805_2012Metric_Pad1.20x1.40mm_HandSolder, symbol Device:R
- added R46: 1k, Resistor_SMD:R_0805_2012Metric_Pad1.20x1.40mm_HandSolder, symbol Device:R
- added R48: k1, Resistor_SMD:R_0201_0603Metric, symbol Device:R
- added R5: M1, Resistor_SMD:R_0805_2012Metric_Pad1.20x1.40mm_HandSolder, symbol Device:R
- added R8: 220k, Resistor_SMD:R_0201_0603Metric, symbol Device:R
- added SW2: SW_SPST, liebler_MECH:KCD1-11-2P, symbol Switch:SW_SPST
- added SW3: 12V/20V, liebler_MECH:SW_SPDT_PCM12_handsolder, symbol liebler_MECH:SW_SPDT_with_Case
- added SW4: RESET, liebler_MECH:Button_2x4x3,5_handsolder, symbol Switch:SW_Push
- added TP1: T24V, TestPoint:TestPoint_THTPad_D1.5mm_Drill0.7mm, symbol Connector:TestPoint
- added TP2: SHAKE, TestPoint:TestPoint_THTPad_D1.5mm_Drill0.7mm, symbol Connector:TestPoint
- added TP3: NTC, TestPoint:TestPoint_THTPad_D1.5mm_Drill0.7mm, symbol Connector:TestPoint
- added TP4: T12+, TestPoint:TestPoint_THTPad_D1.5mm_Drill0.7mm, symbol Connector:TestPoint
- added U1: ~, Package_DFN_QFN:DFN-6-1EP_2x2mm_P0.65mm_EP1.01x1.7mm, symbol liebler_SEMICONDUCTORS:HUSB237
- added U10: DS18B20, Package_TO_SOT_THT:TO-92L_HandSolder, symbol Sensor_Temperature:DS18B20
- added U11: ESP32-S3-WROOM-1, Espressif:ESP32-S3-WROOM-1, symbol RF_Module:ESP32-S3-WROOM-1
- added U2: TPS54202DDC, Package_TO_SOT_SMD:SOT-23-6_Handsoldering, symbol Regulator_Switching:TPS54202DDC
- added U3: 74AHCT1G125, Package_TO_SOT_SMD:SOT-353_SC-70-5_Handsoldering, symbol 74xGxx:74AHCT1G125
- added U4: AMS1117-3.3, liebler_SEMICONDUCTORS:SOT-223-3_TabPin2_HANDSOLDER, symbol Regulator_Linear:AMS1117-3.3
- added U5: OPA336Nx, Package_TO_SOT_SMD:SOT-23-5, symbol Amplifier_Operational:OPA336Nx
- added X1: Display_P169H002-CTP, liebler_OPTO:Display_P169H002-CTP, symbol liebler_OPTO:Display_P169H002-CTP
- J2: value Conn_01x05 -> IRON
- R14, R15: footprint Resistor_SMD:R_0402_1005Metric -> Resistor_SMD:R_0201_0603Metric
- R16: value 5k1 -> 1k; footprint Resistor_SMD:R_0402_1005Metric -> Resistor_SMD:R_0805_2012Metric
- SW1: symbol liebler_SWITCHES:Rotary_Encoder_Switch_with_Mountingpoint -> Device:RotaryEncoder_Switch_MP
Connections:
- net GND: now also D1.4 (VSS), D2.4 (VSS), D3.4 (VSS), D4.4 (VSS), D5.4 (VSS), D6.4 (VSS), D7.4 (VSS), D8.4 (VSS), J1.2, J2.3 (Pin_3), J2.4 (Pin_4), SW1.C, SW1.MP, SW1.S1, C1.1, C10.2, C11.2, C12.2, C13.2, C14.2, C15.2, C16.2, C17.2, C19.2, C2.1, C20.1, C21.2, C22.2, C23.2, C24.2, C25.2, C26.2, C27.2, C28.2, C29.2, C30.2, C31.2, C32.1, C5.2, C6.2, C7.2, C8.2, C9.2, D12.1 (K), J3.A1 (GND), J3.A12 (GND), J3.B1 (GND), J3.B12 (GND), J3.S1 (SHIELD), J32.4 (Pin_4), J5.5 (Pin_5), Q1.2 (E), Q3.2 (E), Q4.2 (E), R10.1, R21.1, R4.1, R7.1, SW3.CASE, SW4.2, U1.7 (GND), U10.1 (GND), U11.1 (GND), U11.40 (GND), U11.41 (GND), U2.1 (GND), U3.1, U3.3 (GND), U4.1 (GND), U5.2 (V-), X1.1 (GND), X1.12 (GND), X1.18 (GND), X1.5 (GND), X1.6 (GND); no longer R16.2
- net USB+: now also U11.14 (USB_D+)
- net USB-: now also U11.13 (USB_D-)
- net +5V: now reaches D4.2 (VDD)
- net +5V: now also D1.2 (VDD), D2.2 (VDD), D3.2 (VDD), D5.2 (VDD), D6.2 (VDD), D7.2 (VDD), D8.2 (VDD), C10.1, C21.1, C22.1, C23.1, C24.1, C26.1, C27.1, C28.1, C29.1, C4.2, C5.1, C6.1, C7.1, C9.1, L1.1, R2.1, U3.5 (VCC), U4.3 (VI)
- net at R16.1: now also D11.1 (K), Q2.4 (G), Q3.3 (C)
- net at J1.1: now also D13.2 (A)
- net at D1.1 (DIN): now also U3.4
- net VBUS_5V: now reaches J6.A4 (VBUS), J6.A9 (VBUS), J6.B4 (VBUS), J6.B9 (VBUS)
- net VBUS_5V: now also R23.2
- net ROT_A: now reaches SW1.A
- net ROT_A: now also C31.1, R18.1, U11.7 (IO7)
- net ROT_B: now reaches SW1.B
- net ROT_B: now also C30.1, R19.1, U11.11 (IO18)
- net IRON_SHAKE: now reaches J2.1 (Pin_1)
- net IRON_SHAKE: now also R12.1, R13.2, TP2.1
- net IRON_NTC: now reaches J2.2 (Pin_2)
- net IRON_NTC: now also R25.1, R27.1, TP3.1
- net IRON_T12+: now reaches J2.5 (Pin_5)
- net IRON_T12+: now also C14.1, C18.2, D11.2 (A), Q2.1 (S), Q2.2 (S), Q2.3 (S), R11.1, TP4.1
- new net: R10.2, R8.2, U5.4 (-)
- new net: R48.1, SW4.1
- new net: BZ1.N (-), R30.1
- new net: C13.1, D12.2 (A), R11.2, U5.3 (+)
- new net: R26.2, X1.2 (LEDK)
- new net: Q4.1 (B), R3.1
- new net: R1.1, R4.2
- new net: J3.A5 (CC1), U1.1 (CC1)
- new net: C19.1, D9.2 (A), J3.A4 (VBUS), J3.A9 (VBUS), J3.B4 (VBUS), J3.B9 (VBUS), U1.2 (VBUS)
- new net: JP1.1 (A), SW3.2 (B), U1.3 (VSET)
- new net: J3.A6 (D+), J3.B6 (D+), U1.4 (D+)
- new net: J3.A7 (D-), J3.B7 (D-), U1.5 (D-)
- new net: J3.B5 (CC2), U1.6 (CC2)
- new net: Q1.3 (C), R30.2
- new net: C18.1, D10.1 (K), R16.2
- new net: C20.2, JP1.2 (B), SW3.3 (C)
- new net: R22.2, R23.1
- new net: Q3.1 (B), R17.1
- new net: Q4.3 (C), R26.1
- new net: Q1.1 (B), R6.1
- new net +24V: C1.2, C2.2, D10.2 (A), Q2.5 (D), R5.2, SW2.2 (B), TP1.1, U2.3 (VIN)
- new net +3V3: BZ1.P (+), C11.1, C12.1, C15.1, C16.1, C17.1, C8.1, J32.2 (Pin_2), J5.1 (Pin_1), R12.2, R18.2, R19.2, R20.1, R24.2, R27.2, R28.2, R29.2, R46.2, R47.2, R9.2, U10.3 (V_{DD}), U11.2 (3V3), U4.2 (VO), U5.5 (V+), X1.17 (VCC), X1.3 (VCC), X1.4 (IOVCC)
- new net BOOT: C3.1, U2.6 (BOOT)
- new net BUZZER: R6.2, U11.18 (IO10)
- new net EXT_SCL: J5.3 (Pin_3), R28.1, U11.8 (IO15)
- new net EXT_SDA: J5.4 (Pin_4), R29.1, U11.9 (IO16)
- new net FB: C4.1, R1.2, R2.2, U2.4 (FB)
- new net IRON_MOSFET: R17.2, U11.34 (IO41)
- new net IRON_SHAKE_I: R13.1, U11.33 (IO40)
- new net IRON_TEMP_NTC: R25.2, U11.38 (IO2)
- new net IRON_TEMP_THERM: R8.1, U11.39 (IO1), U5.1
- new net LCD_BL: R3.2, U11.26 (IO45)
- new net LCD_CS: U11.20 (IO12), X1.8 (CS)
- new net LCD_DAT: U11.22 (IO14), X1.10 (SDA)
- new net LCD_RES: U11.23 (IO21), X1.11 (RESET)
- new net LCD_RS: U11.19 (IO11), X1.7 (RS)
- new net LCD_SCK: U11.21 (IO13), X1.9 (SCK)
- new net Onewire: J5.2 (Pin_2), R46.1, U10.2 (DQ), U11.4 (IO4)
- new net PROG_EN: C25.1, J32.1 (Pin_1), R47.1, R48.2, U11.3 (EN)
- new net PROG_IO0: C32.2, J32.6 (Pin_6), R20.2, SW1.S2, U11.27 (IO0)
- new net PROG_RX: J32.5 (Pin_5), U11.36 (RXD0)
- new net PROG_TX: J32.3 (Pin_3), U11.37 (TXD0)
- new net PSU_SW: C3.2, L1.2, U2.2 (SW)
- new net RGB_LED: U11.15 (IO3), U3.2
- new net TP_IRQ: U11.32 (IO39), X1.16 (TP_TINT)
- new net TP_RST: U11.31 (IO38), X1.15 (TP_TRST)
- new net TP_SCL: R9.1, U11.24 (IO47), X1.13 (TP_SCL)
- new net TP_SDA: R24.1, U11.25 (IO48), X1.14 (TP_SDA)
- new net VBUS: D13.1 (K), D9.1 (K), SW2.1 (A)
- new net VBUS_5V_SENSE: R21.2, R22.1, U11.12 (IO8)
- new net VBUS_MEASURE: R5.1, R7.2, U11.17 (IO9)
- no-connect marks 2 -> 10
Other:
- note added: "5V->3,3V + microUSV"
- note added: "Buzzer"
- note added: "CPU"
- note added: "GPIO0: PU, aber jederzeit PD GPIO3: JTAG -> Floating GPIO45: Voltage ->PD GPIO46: Logging ->PD"
- note added: "Own Measurement 2025-09-11: 10,4k @ 23°C"
- note added: "PROG"
- note added: "Reset / Boot"
- note added: "open=12V, 22nF=20V"
- moved on the sheet: J2

Commit message: Various Updates
Parts:
- removed C20: 22n, Capacitor_SMD:C_0201_0603Metric, symbol Device:C
- removed JP1: 20V, Jumper:SolderJumper-2_P1.3mm_Open_RoundedPad1.0x1.5mm, symbol Jumper:Jumper_2_Open
- removed SW3: 12V/20V, liebler_MECH:SW_SPDT_PCM12_handsolder, symbol liebler_MECH:SW_SPDT_with_Case
- removed U1: ~, Package_DFN_QFN:DFN-6-1EP_2x2mm_P0.65mm_EP1.01x1.7mm, symbol liebler_SEMICONDUCTORS:HUSB237
- added R31: M1, Resistor_SMD:R_0201_0603Metric, symbol Device:R
- added R32, R33: 10k, Resistor_SMD:R_0201_0603Metric, symbol Device:R
- added U6: ~, Package_DFN_QFN:Texas_DSQ0010A_WSON-10-1EP_2x2mm_P0.4mm_EP0.9x1.5mm_ThermalVias, symbol liebler_SEMICONDUCTORS:CH224Q
Connections:
- net GND: now also R33.1, U6.11 (PAD_/_GND)
- net IRON_MOSFET: now also U11.33 (IO40); no longer U11.34 (IO41)
- net IRON_SHAKE_I: now also U11.34 (IO41); no longer U11.33 (IO40)
- net TP_SCL: now also U6.2 (CFG2/SCL)
- net TP_SDA: now also U6.3 (CFG3/SDA)
- net at J3.A5 (CC1): now also U6.7 (CC1)
- net at C19.1, D9.2 (A), J3.A4 (VBUS)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: now also U6.1 (VHV), U6.8 (VBUS)
- net at J3.A6 (D+), J3.B6 (D+): now also U6.4 (DP)
- net at J3.A7 (D-), J3.B7 (D-): now also U6.5 (DM)
- net at J3.B5 (CC2): now also U6.6 (CC2)
- new net: R32.1, R33.2
- new net: R31.2, R32.2
- new net: R31.1, U6.9 (CFG1)
Other:
- note removed: "open=12V, 22nF=20V"
- moved on the sheet: C19, D9, J3
