File: soldering_station.kicad_pcb (KiCad board)
At the start: 2 copper layers, 100 x 43 mm, 17 parts, among them J1 Barrel_Jack_Switch, J2 Conn_01x05, J6 USB, SW1 Rotary_Encoder_Switch_with_Mo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, U1 2.4inch_ST7789V_LCD

Commit message: WIP
Parts:
- D2, D3, D4, D5, D6, D7, D8: moved to B.Cu
- moved D1 88.2 mm to (140.0, 30.0)
- moved D2 74.2 mm to (128.6, 30.0)
- moved D8 70.4 mm to (60.0, 30.0)
- moved D3 68.6 mm to (117.1, 30.0)
- moved D7 65.9 mm to (71.4, 30.0)
- moved D4 64.7 mm to (105.7, 30.0)
- moved D6 63.3 mm to (82.9, 30.0)
- moved D5 62.9 mm to (94.3, 30.0)

Commit message: Ready for review
Parts:
- removed R54: 3k3, Resistor_SMD:R_0402_1005Metric
- added BZ1: Buzzer, liebler_MECH:XDCR_CMT-7525-80-SMT-TR_handsolder, B.Cu at (95.3, 61.4)
- added C1: u1/35V, Capacitor_SMD:C_0805_2012Metric, B.Cu at (135.3, 64.3)
- added C10: u1, Capacitor_SMD:C_0201_0603Metric, B.Cu at (137.7, 44.4)
- added C11: u1, Capacitor_SMD:C_0201_0603Metric, B.Cu at (147.1, 44.5)
- added C12: 10u, Capacitor_SMD:C_0603_1608Metric, B.Cu at (145.8, 44.6)
- added C13: 2n2, Capacitor_SMD:C_0201_0603Metric, B.Cu at (57.3, 46.0)
- added C14: 1u, Resistor_SMD:R_0402_1005Metric, B.Cu at (57.5, 47.3)
- added C15: u1, Capacitor_SMD:C_0201_0603Metric, B.Cu at (120.1, 40.4)
- added C16: 22u, Capacitor_SMD:C_0603_1608Metric, B.Cu at (121.4, 40.3)
- added C17: 1u, Resistor_SMD:R_0402_1005Metric, B.Cu at (83.0, 52.5)
- added C18: 10u/35V, Capacitor_SMD:C_0603_1608Metric, B.Cu at (60.7, 47.6)
- added C19: 1u, Capacitor_SMD:C_0201_0603Metric, B.Cu at (60.2, 52.4)
- added C2: 10u/35V, Capacitor_SMD:C_1206_3216Metric, B.Cu at (131.3, 63.1)
- added C20: 22n, Capacitor_SMD:C_0201_0603Metric, B.Cu at (70.4, 64.9)
- added C21: u1, Capacitor_SMD:C_0201_0603Metric, B.Cu at (129.7, 65.0)
- added C22: u1, Capacitor_SMD:C_0201_0603Metric, B.Cu at (121.5, 64.7)
- added C23: u1, Capacitor_SMD:C_0201_0603Metric, B.Cu at (113.1, 64.8)
- added C24: u1, Capacitor_SMD:C_0201_0603Metric, B.Cu at (105.2, 64.8)
- added C25: u1, Capacitor_SMD:C_0201_0603Metric, B.Cu at (87.1, 35.8)
- added C26: u1, Capacitor_SMD:C_0201_0603Metric, B.Cu at (92.4, 66.1)
- added C27: u1, Capacitor_SMD:C_0201_0603Metric, B.Cu at (87.8, 64.8)
- added C28: u1, Capacitor_SMD:C_0201_0603Metric, B.Cu at (81.7, 64.7)
- added C29: u1, Capacitor_SMD:C_0201_0603Metric, B.Cu at (71.7, 64.7)
- added C3: u1/16V, Capacitor_SMD:C_0201_0603Metric, B.Cu at (130.6, 57.5)
- added C30: 10n, Capacitor_SMD:C_0201_0603Metric, B.Cu at (126.6, 53.1)
- added C31: 10n, Capacitor_SMD:C_0201_0603Metric, B.Cu at (125.1, 45.8)
- added C32: 10n, Capacitor_SMD:C_0201_0603Metric, B.Cu at (99.2, 55.7)
- added C4: 56p, Capacitor_SMD:C_0201_0603Metric, B.Cu at (129.5, 57.9)
- added C5: 22u, Resistor_SMD:R_0805_2012Metric_Pad1.20x1.40mm_HandSolder, B.Cu at (144.5, 59.5)
- added C6: 22u, Resistor_SMD:R_0805_2012Metric_Pad1.20x1.40mm_HandSolder, B.Cu at (144.5, 57.6)
- added C7: u1, Capacitor_SMD:C_0201_0603Metric, B.Cu at (116.1, 64.2)
- added C8: u1, Capacitor_SMD:C_0201_0603Metric, B.Cu at (56.4, 41.6)
- added C9: 10u, Capacitor_SMD:C_0603_1608Metric, B.Cu at (136.6, 44.4)
- added D10: ~, liebler_SEMICONDUCTORS:D_SOD-123_handsolder, B.Cu at (62.1, 44.5)
- added D11: 18V, liebler_SEMICONDUCTORS:D_SOD-123_handsolder, B.Cu at (63.2, 50.4)
- added D12: LED, LED_SMD:LED_0805_2012Metric_Pad1.15x1.40mm_HandSolder, F.Cu at (58.1, 53.8)
- added D13: D_Schottky, Diode_SMD:D_SMA, B.Cu at (68.6, 59.9)
- added D9: D_Schottky, Diode_SMD:D_SMA, B.Cu at (55.4, 54.9)
- added G***: LOGO, LOGO, B.Cu at (76.7, 52.9)
- added H1: MountingHole, MountingHole:MountingHole_3.2mm_M3, F.Cu at (146.0, 50.0)
- added H2: MountingHole, MountingHole:MountingHole_3.2mm_M3, F.Cu at (54.0, 50.0)
- added J3: USB, liebler_CONN:GT-USB-7051A, B.Cu at (60.6, 59.0)
- added J32: PROG, Connector_PinHeader_1.27mm:PinHeader_2x03_P1.27mm_Vertical_SMD, B.Cu at (82.0, 39.6)
- added J5: EXT, Connector_PinHeader_2.54mm:PinHeader_1x05_P2.54mm_Vertical, B.Cu at (121.5, 43.6)
- added JP1: 20V, Jumper:SolderJumper-2_P1.3mm_Open_RoundedPad1.0x1.5mm, B.Cu at (69.2, 62.9)
- added L1: 10uH, Inductor_SMD:L_Abracon_ASPI-0630LR, B.Cu at (138.2, 59.7)
- added Q1: BC847, Package_TO_SOT_SMD:SOT-23, B.Cu at (108.1, 64.1)
- added Q2: Q_PMOS_GDS, Package_DFN_QFN:PQFN-8-EP_6x5mm_P1.27mm_Generic, B.Cu at (67.8, 46.1)
- added Q3: MMBT2222A, Package_TO_SOT_SMD:SOT-23, B.Cu at (76.2, 43.8)
- added Q4: BC847, Package_TO_SOT_SMD:SOT-23_Handsoldering, B.Cu at (83.9, 62.7)
- added R1: 10k, Resistor_SMD:R_0201_0603Metric, B.Cu at (128.8, 56.2)
- added R10: 1k, Resistor_SMD:R_0201_0603Metric, B.Cu at (54.6, 44.9)
- added R11: 4k7, Resistor_SMD:R_0805_2012Metric_Pad1.20x1.40mm_HandSolder, B.Cu at (59.0, 47.6)
- added R12: 3k3, Resistor_SMD:R_0201_0603Metric, B.Cu at (71.4, 47.8)
- added R13: 3k3, Resistor_SMD:R_0201_0603Metric, B.Cu at (84.9, 43.2)
- added R17: 10k, Resistor_SMD:R_0201_0603Metric, B.Cu at (84.9, 42.5)
- added R18: 3k3, Resistor_SMD:R_0201_0603Metric, B.Cu at (126.6, 47.5)
- added R19: 3k3, Resistor_SMD:R_0201_0603Metric, B.Cu at (126.6, 52.4)
- added R2: M1, Resistor_SMD:R_0201_0603Metric, B.Cu at (129.5, 57.2)
- added R20: 3k3, Resistor_SMD:R_0201_0603Metric, B.Cu at (99.2, 56.4)
- added R21: 10k, Resistor_SMD:R_0201_0603Metric, B.Cu at (125.1, 54.6)
- added R22: 10k, Resistor_SMD:R_0201_0603Metric, B.Cu at (126.2, 54.9)
- added R23: 10k, Resistor_SMD:R_0201_0603Metric, B.Cu at (126.2, 55.7)
- added R24: 3k3, Resistor_SMD:R_0201_0603Metric, B.Cu at (82.6, 47.5)
- added R25: 5k1, Resistor_SMD:R_0201_0603Metric, B.Cu at (77.2, 38.0)
- added R26: 22R, Resistor_SMD:R_0805_2012Metric_Pad1.20x1.40mm_HandSolder, B.Cu at (82.9, 57.3)
- added R27: 10k, Resistor_SMD:R_0201_0603Metric, B.Cu at (72.2, 47.8)
- added R28: 3k3, Resistor_SMD:R_0201_0603Metric, B.Cu at (126.6, 48.9)
- added R29: 3k3, Resistor_SMD:R_0201_0603Metric, B.Cu at (126.6, 51.1)
- added R3: 1k, Resistor_SMD:R_0201_0603Metric, B.Cu at (87.6, 62.9)
- added R30: 22R, Resistor_SMD:R_0805_2012Metric_Pad1.20x1.40mm_HandSolder, B.Cu at (102.9, 64.6)
- added R4: 3k3, Resistor_SMD:R_0201_0603Metric, B.Cu at (127.7, 55.2)
- added R46: 1k, Resistor_SMD:R_0805_2012Metric_Pad1.20x1.40mm_HandSolder, B.Cu at (132.1, 40.8)
- added R47: 10k, Resistor_SMD:R_0201_0603Metric, B.Cu at (86.7, 39.3)
- added R48: k1, Resistor_SMD:R_0201_0603Metric, B.Cu at (85.4, 35.8)
- added R5: M1, Resistor_SMD:R_0805_2012Metric_Pad1.20x1.40mm_HandSolder, B.Cu at (114.4, 61.7)
- added R6: 1k, Resistor_SMD:R_0201_0603Metric, B.Cu at (110.9, 60.8)
- added R7: 10k, Resistor_SMD:R_0201_0603Metric, B.Cu at (114.7, 59.1)
- added R8: 220k, Resistor_SMD:R_0201_0603Metric, B.Cu at (54.6, 43.5)
- added R9: 3k3, Resistor_SMD:R_0201_0603Metric, B.Cu at (82.6, 48.3)
- added SW2: SW_SPST, liebler_MECH:KCD1-11-2P, F.Cu at (68.0, 39.0)
- added SW3: 12V/20V, liebler_MECH:SW_SPDT_PCM12_handsolder, F.Cu at (68.0, 64.3)
- added SW4: RESET, liebler_MECH:Button_2x4x3,5_handsolder, B.Cu at (75.2, 34.1)
- added TP1: T24V, TestPoint:TestPoint_THTPad_D1.5mm_Drill0.7mm, B.Cu at (70.6, 39.0)
- added TP2: SHAKE, TestPoint:TestPoint_THTPad_D1.5mm_Drill0.7mm, B.Cu at (79.4, 48.1)
- added TP3: NTC, TestPoint:TestPoint_THTPad_D1.5mm_Drill0.7mm, B.Cu at (72.7, 50.2)
- added TP4: T12+, TestPoint:TestPoint_THTPad_D1.5mm_Drill0.7mm, B.Cu at (61.3, 49.6)
- added U10: DS18B20, Package_TO_SOT_THT:TO-92L_HandSolder, F.Cu at (127.0, 42.6)
- added U11: ESP32-S3-WROOM-1, Espressif:ESP32-S3-WROOM-1, B.Cu at (109.8, 48.1)
- added U2: TPS54202DDC, Package_TO_SOT_SMD:SOT-23-6_Handsoldering, B.Cu at (131.3, 60.1)
- added U3: 74AHCT1G125, Package_TO_SOT_SMD:SOT-353_SC-70-5_Handsoldering, B.Cu at (116.8, 61.1)
- added U4: AMS1117-3.3, liebler_SEMICONDUCTORS:SOT-223-3_TabPin2_HANDSOLDER, B.Cu at (141.6, 41.5)
- added U5: OPA336Nx, Package_TO_SOT_SMD:SOT-23-5, B.Cu at (57.0, 43.7)
- added X1: Display_P169H002-CTP, liebler_OPTO:Display_P169H002-CTP, B.Cu at (86.0, 50.0)
- J2: value Conn_01x05 -> IRON
- R14, R15: footprint Resistor_SMD:R_0402_1005Metric -> Resistor_SMD:R_0201_0603Metric; moved to B.Cu
- R16: value 5k1 -> 1k; footprint Resistor_SMD:R_0402_1005Metric -> Resistor_SMD:R_0805_2012Metric; moved to B.Cu
- U1: value 2.4inch_ST7789V_LCD -> ~; footprint liebler_OPTO:2,4zoll lcd tft touch -> Package_DFN_QFN:DFN-6-1EP_2x2mm_P0.65mm_EP1.01x1.7mm; moved to B.Cu
- moved R15 101.3 mm to (124.3, 61.7)
- moved R14 100.9 mm to (124.8, 56.3), turned to 180 degrees
- moved J6 65.1 mm to (124.2, 59.0), turned to 180 degrees
- moved J1 63.6 mm to (76.7, 59.0), turned to 180 degrees
- moved U1 43.5 mm to (60.2, 54.7)
- moved D1 37.9 mm to (129.5, 66.4), turned to 180 degrees
- moved D8 37.9 mm to (70.5, 66.4), turned to 180 degrees
- moved R16 37.8 mm to (63.2, 46.6), turned to 180 degrees
- moved D2 37.2 mm to (121.1, 66.4), turned to 180 degrees
- moved D7 37.2 mm to (78.9, 66.4), turned to 180 degrees
- moved D3 36.7 mm to (112.6, 66.4), turned to 180 degrees
- moved D6 36.7 mm to (87.4, 66.4), turned to 180 degrees
- moved D4 36.4 mm to (104.2, 66.4), turned to 180 degrees
- moved D5 36.4 mm to (95.8, 66.4), turned to 180 degrees
- moved J2 9.08 mm to (68.0, 53.8)
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Connections:
- net Net-(J6-VBUS-PadA4) renamed VBUS_5V
- D1 pad 1: unconnected-(D1-DIN-Pad1) -> Net-(D1-DIN)
- D1 pad 2: unconnected-(D1-VDD-Pad2) -> +5V
- D1 pad 4: unconnected-(D1-VSS-Pad4) -> GND
- D2 pad 2: unconnected-(D2-VDD-Pad2) -> +5V
- D2 pad 4: unconnected-(D2-VSS-Pad4) -> GND
- D3 pad 2: unconnected-(D3-VDD-Pad2) -> +5V
- D3 pad 4: unconnected-(D3-VSS-Pad4) -> GND
- D4 pad 2: unconnected-(D4-VDD-Pad2) -> +5V
- D4 pad 4: unconnected-(D4-VSS-Pad4) -> GND
- D5 pad 2: unconnected-(D5-VDD-Pad2) -> +5V
- D5 pad 4: unconnected-(D5-VSS-Pad4) -> GND
- D6 pad 2: unconnected-(D6-VDD-Pad2) -> +5V
- D6 pad 4: unconnected-(D6-VSS-Pad4) -> GND
- D7 pad 2: unconnected-(D7-VDD-Pad2) -> +5V
- D7 pad 4: unconnected-(D7-VSS-Pad4) -> GND
- D8 pad 2: unconnected-(D8-VDD-Pad2) -> +5V
- D8 pad 4: unconnected-(D8-VSS-Pad4) -> GND
- J1 pad 1: unconnected-(J1-Pad1) -> Net-(D13-A)
- J1 pad 2: unconnected-(J1-Pad2) -> GND
- J2 pad 1: unconnected-(J2-Pin_1-Pad1) -> IRON_SHAKE
- J2 pad 2: unconnected-(J2-Pin_2-Pad2) -> IRON_NTC
- J2 pad 3: unconnected-(J2-Pin_3-Pad3) -> GND
- J2 pad 4: unconnected-(J2-Pin_4-Pad4) -> GND
- J2 pad 5: unconnected-(J2-Pin_5-Pad5) -> IRON_T12+
- R16 pad 2: GND -> Net-(D10-K)
- SW1 pad A: unconnected-(SW1-PadA) -> ROT_A
- SW1 pad B: unconnected-(SW1-PadB) -> ROT_B
- SW1 pad C: unconnected-(SW1-PadC) -> GND
- SW1 pad MP: unconnected-(SW1-PadMP) -> GND
- SW1 pad S1: (no net) -> GND
- SW1 pad S2: (no net) -> PROG_IO0
- U1 pad 1: unconnected-(U1-GND-Pad1) -> Net-(J3-CC1)
- U1 pad 2: unconnected-(U1-nRESET-Pad2) -> Net-(D9-A)
- U1 pad 3: unconnected-(U1-SCL-Pad3) -> Net-(JP1-A)
- U1 pad 4: unconnected-(U1-DC-Pad4) -> Net-(U1-D+)
- U1 pad 5: unconnected-(U1-CSX-Pad5) -> Net-(U1-D-)
- U1 pad 6: unconnected-(U1-SDI-Pad6) -> Net-(J3-CC2)
- U1 pad 7: unconnected-(U1-SDO-Pad7) -> GND
Routing:
- net +3V3: track 0.00 -> 146.8 mm, vias 0 -> 43
- net +5V: track 0.00 -> 145.9 mm, vias 0 -> 9
- net +24V: track 0.00 -> 83.4 mm, vias 0 -> 3
- net PROG_IO0: track 0.00 -> 78.5 mm, vias 0 -> 4
- net GND: track 0.00 -> 63.8 mm, vias 0 -> 175
- net IRON_TEMP_THERM: track 0.00 -> 55.9 mm
- net PROG_EN: track 0.00 -> 41.4 mm, vias 0 -> 4
- net LCD_RS: track 0.00 -> 40.7 mm
- net LCD_CS: track 0.00 -> 38.4 mm
- net LCD_SCK: track 0.00 -> 37.8 mm
- net LCD_DAT: track 0.00 -> 35.5 mm
- net LCD_RES: track 0.00 -> 34.4 mm
- net TP_SCL: track 0.00 -> 34.2 mm
- net TP_SDA: track 0.00 -> 32.8 mm
- net Net-(D9-A): track 0.00 -> 26.8 mm
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- added copper zone on B.Cu, net +24V
- added copper zone on B.Cu, net +3V3
- added copper zone on F.Cu, net +3V3
- added copper zone on B.Cu, net GND
- added copper zone on F.Cu, net GND
- added copper zone on B.Cu, net IRON_T12+
Other:
- board size 100 x 43 mm -> 100 x 36 mm
- board text added: "12V/20V"
- board text added: "1Wire"
- board text added: "24V"
- board text added: "3V3"
- board text added: "ENCODER PUSH=BOOT"
- board text added: "ESP PROG"
- board text added: "GND"
- board text added: "IRON"
- board text added: "NTC"
- board text added: "OFF"
- board text added: "ON"
- board text added: "RESET"
- board text added: "ROOM TEMP"
- board text added: "SCL"
- board text added: "SDA"
- board text added: "SHAKE"
- board text added: "T12+"
- board text added: "USB CTRL"
- board text added: "USB PD"

Commit message: Various Updates
Parts:
- removed C20: 22n, Capacitor_SMD:C_0201_0603Metric
- removed JP1: 20V, Jumper:SolderJumper-2_P1.3mm_Open_RoundedPad1.0x1.5mm
- removed SW3: 12V/20V, liebler_MECH:SW_SPDT_PCM12_handsolder
- removed U1: ~, Package_DFN_QFN:DFN-6-1EP_2x2mm_P0.65mm_EP1.01x1.7mm
- added R31: M1, Resistor_SMD:R_0201_0603Metric, B.Cu at (58.9, 52.1)
- added R32: 10k, Resistor_SMD:R_0201_0603Metric, B.Cu at (58.5, 51.0)
- added R33: 10k, Resistor_SMD:R_0201_0603Metric, B.Cu at (58.1, 52.1)
- added U6: ~, Package_DFN_QFN:Texas_DSQ0010A_WSON-10-1EP_2x2mm_P0.4mm_EP0.9x1.5mm_ThermalVias, B.Cu at (60.6, 54.2)
- moved TP3 10.2 mm to (76.2, 40.5)
- moved R13 9.90 mm to (75.0, 42.2)
- moved TP2 8.09 mm to (72.5, 52.4)
- moved R17 5.55 mm to (79.3, 42.7)
- moved R9 3.38 mm to (79.5, 47.0), turned to 90 degrees
- moved G*** 2.87 mm to (76.5, 50.0)
- moved R26 2.80 mm to (82.4, 60.0)
- moved R24 2.41 mm to (80.3, 47.0), turned to 90 degrees
- moved C17 2.15 mm to (80.8, 52.5)
- moved X1 2.05 mm to (84.0, 50.0)
- moved C19 1.43 mm to (61.6, 52.1)
- moved Q4 1.32 mm to (84.8, 63.7), turned to 180 degrees
- moved R3 0.72 mm to (88.2, 62.6)
- moved R27 0.63 mm to (71.8, 48.4)
- moved R12 0.60 mm to (71.2, 48.4)
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Connections:
- U11 pad 33: IRON_SHAKE_I -> IRON_MOSFET
- U11 pad 34: IRON_MOSFET -> IRON_SHAKE_I
Routing:
- net TP_SCL: track 34.2 -> 60.5 mm
- net TP_SDA: track 32.8 -> 58.9 mm, vias 0 -> 2
- net +3V3: track 146.8 -> 172.1 mm
- net Net-(JP1-A): track 15.0 -> 0.00 mm, vias 2 -> 0
- net IRON_SHAKE_I: track 19.2 -> 29.4 mm
- net IRON_MOSFET: track 18.5 -> 25.6 mm
- net Net-(Q3-B): track 7.59 -> 1.43 mm
- net IRON_SHAKE: track 23.1 -> 18.4 mm, vias 1 -> 0
- net Net-(D9-A): track 26.8 -> 31.2 mm, vias 0 -> 3
- net LCD_BL: track 21.9 -> 18.7 mm
- net Net-(X1-LEDK): track 3.63 -> 6.82 mm
- net Net-(JP1-B): track 3.11 -> 0.00 mm, vias 1 -> 0
- net Net-(J3-CC2): track 6.09 -> 3.56 mm
- net Net-(U6-DP): track 4.13 -> 6.53 mm
- net TP_RST: track 24.2 -> 26.3 mm
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Other:
- outline, holes or cut-outs redrawn

Commit message: Layout improvements
Routing:
- net +3V3: track 172.1 -> 150.7 mm
- net LCD_SCK: track 37.5 -> 38.5 mm
- net LCD_RS: track 40.0 -> 40.8 mm
- net LCD_CS: track 38.7 -> 39.6 mm
